Commit message: Adding simulated ensenso.

File: sr_camera_launch/description/ensenso.gazebo.xacro (robot description, xacro)
@@ -2,5 +2,5 @@
 <robot xmlns:xacro="http://ros.org/wiki/xacro">
   <xacro:macro name="sim_ensenso_sensor" params="camera_name">
-    <gazebo reference="${camera_name}_depth">
+    <gazebo reference="${camera_name}_depth_frame">
       <sensor type="depth" name="${camera_name}_depth">
         <always_on>true</always_on>
@@ -19,13 +19,13 @@
         </camera>
         <plugin name="kinect_camera_controller" filename="libgazebo_ros_openni_kinect.so">
-          <cameraName>${camera_name}</cameraName>
+          <cameraName>/camera</cameraName>
           <alwaysOn>true</alwaysOn>
           <updateRate>10.0</updateRate>
-          <imageTopicName>rgb/image</imageTopicName>
+          <imageTopicName>depth_registered/rgb/image</imageTopicName>
           <depthImageTopicName>depth_registered/image_raw</depthImageTopicName>
           <pointCloudTopicName>depth_registered/points</pointCloudTopicName>
-          <cameraInfoTopicName>rgb/camera_info</cameraInfoTopicName>
+          <cameraInfoTopicName>depth_registered/rgb/camera_info</cameraInfoTopicName>
           <depthImageCameraInfoTopicName>depth_registered/camera_info</depthImageCameraInfoTopicName>
-          <frameName>${camera_name}_depth_frame</frameName>
+          <frameName>${camera_name}_left_ir_optical_frame</frameName>
           <baseline>0.2</baseline>
           <distortion_k1>0.0</distortion_k1>
@@ -38,5 +38,5 @@
       </sensor>
     </gazebo>
-    <gazebo reference="${camera_name}_rgb">
+    <gazebo reference="${camera_name}_rgb_frame">
       <sensor type="camera" name="${camera_name}_rgb">
         <always_on>true</always_on>
@@ -50,25 +50,86 @@
           </image>
           <clip>
-            <near>0.4</near>
-            <far>8.0</far>
+            <near>0.1</near>
+            <far>50.0</far>
           </clip>
         </camera>
-        <plugin name="kinect_camera_controller" filename="libgazebo_ros_openni_kinect.so">
-          <cameraName>${camera_name}</cameraName>
+        <plugin name="camera_controller" filename="libgazebo_ros_camera.so">
+          <cameraName>camera/rgb</cameraName>
           <alwaysOn>true</alwaysOn>
           <updateRate>10.0</updateRate>
-          <imageTopicName>rgb/image</imageTopicName>
-          <depthImageTopicName>depth_registered/image_raw</depthImageTopicName>
-          <pointCloudTopicName>depth_registered/points</pointCloudTopicName>
-          <cameraInfoTopicName>rgb/camera_info</cameraInfoTopicName>
-          <depthImageCameraInfoTopicName>depth_registered/camera_info</depthImageCameraInfoTopicName>
-          <frameName>${camera_name}_depth_frame</frameName>
+          <imageTopicName>image</imageTopicName>
+          <cameraInfoTopicName>camera_info</cameraInfoTopicName>
+          <frameName>${camera_name}_rgb_optical_frame</frameName>
           <baseline>0.2</baseline>
-          <distortion_k1>0.0</distortion_k1>
-          <distortion_k2>0.0</distortion_k2>
-          <distortion_k3>0.0</distortion_k3>
+          , , 0.0, 0.0,
+          <distortion_k1>-0.06912065297365189</distortion_k1>
+          <distortion_k2>0.15109966695308685</distortion_k2>
           <distortion_t1>0.0</distortion_t1>
           <distortion_t2>0.0</distortion_t2>
-          <pointCloudCutoff>0.4</pointCloudCutoff>
+          <distortion_k3>-0.17636333405971527</distortion_k3>
+        </plugin>
+      </sensor>
+    </gazebo>
+    <gazebo reference="${camera_name}_left_ir_frame">
+      <sensor type="camera" name="${camera_name}_left_ir">
+        <always_on>true</always_on>
+        <update_rate>60.0</update_rate>
+        <camera>
+          <horizontal_fov>${40.0*M_PI/180.0}</horizontal_fov>
+          <image>
+            <format>L8</format>
+            <width>752</width>
+            <height>480</height>
+          </image>
+          <clip>
+            <near>0.1</near>
+            <far>50.0</far>
+          </clip>
+        </camera>
+        <plugin name="camera_controller" filename="libgazebo_ros_camera.so">
+          <cameraName>camera/ir/left</cameraName>
+          <alwaysOn>true</alwaysOn>
+          <updateRate>10.0</updateRate>
+          <imageTopicName>image</imageTopicName>
+          <cameraInfoTopicName>camera_info</cameraInfoTopicName>
+          <frameName>${camera_name}_left_ir_optical_frame</frameName>
+          <baseline>0.2</baseline>
+          <distortion_k1>-0.5359825420859319</distortion_k1>
+          <distortion_k2>-0.092903692869537</distortion_k2>
+          <distortion_t1>0.000961082680415829</distortion_t1>
+          <distortion_t2>0.0009474949065283347</distortion_t2>
+          <distortion_k3>1.6107857183455494</distortion_k3>
+        </plugin>
+      </sensor>
+    </gazebo>
+    <gazebo reference="${camera_name}_right_ir_frame">
+      <sensor type="camera" name="${camera_name}_right_ir">
+        <always_on>true</always_on>
+        <update_rate>60.0</update_rate>
+        <camera>
+          <horizontal_fov>${40.0*M_PI/180.0}</horizontal_fov>
+          <image>
+            <format>L8</format>
+            <width>752</width>
+            <height>480</height>
+          </image>
+          <clip>
+            <near>0.1</near>
+            <far>50.0</far>
+          </clip>
+        </camera>
+        <plugin name="camera_controller" filename="libgazebo_ros_camera.so">
+          <cameraName>camera/ir/right</cameraName>
+          <alwaysOn>true</alwaysOn>
+          <updateRate>10.0</updateRate>
+          <imageTopicName>image</imageTopicName>
+          <cameraInfoTopicName>camera_info</cameraInfoTopicName>
+          <frameName>${camera_name}_right_ir_optical_frame</frameName>
+          <baseline>0.2</baseline>
+          <distortion_k1>-0.5371060778819661</distortion_k1>
+          <distortion_k2>-0.33074517111569113</distortion_k2>
+          <distortion_t1>0.0003513028055084967</distortion_t1>
+          <distortion_t2>0.0007568502084978531</distortion_t2>
+          <distortion_k3>5.228644677684081</distortion_k3>
         </plugin>
       </sensor>

File: sr_camera_launch/description/ensenso.urdf.xacro (robot description, xacro)
@@ -16,5 +16,5 @@
         <origin xyz="0.0 0.0 0.0" rpy="0 0 0"/>
   	    <geometry>
-  	      <box size="0.07271 0.27794 0.073"/>
+  	      <box size="0.045 0.150 0.045"/>
   	    </geometry>
   	  </collision>
